File: pe/kicad-template/template.kicad_sch (KiCad schematic)
At the start: 0 parts

Commit message: PE SCH and PCB
Started adn finished working on the schematic and now tyring to figure out how the pcb works
Parts:
- added C1: 47uF, Capacitor_SMD:C_1210_3225Metric, symbol Device:C
- added C2: 10uF, Capacitor_SMD:C_1210_3225Metric, symbol Device:C
- added C3: 0.1uF, Capacitor_SMD:C_0603_1608Metric, symbol Device:C
- added L1: 4.7uH, Inductor_SMD:L_Abracon_ASPI-4030S, symbol Device:L
- added R1: 54.9k, Resistor_SMD:R_0805_2012Metric, symbol Device:R
- added R2: 10k, Resistor_SMD:R_0805_2012Metric, symbol Device:R
- added U1: TPS562200, Package_TO_SOT_SMD:SOT-23-6, symbol Regulator_Switching:TPS562200
Connections:
- new net: C3.1, L1.1, U1.2 (SW)
- new net: R1.1, R2.1, U1.4 (VFB)
- new net: C3.2, U1.6 (VBST)
- new net +12V: C2.1, U1.3 (VIN), U1.5 (EN)
- new net GND: C1.2, C2.2, R2.2, U1.1 (GND)
- new net VOUT: C1.1, L1.2, R1.2
