File: pe/kicad-template/template.kicad_pcb (KiCad board)
At the start: 2 copper layers, 7 parts, among them U1 TPS562200

Commit message: PE finished part 3
Finished the pcb, proabbaly gonna chekc it with somone becuase I dont know what the fuck i was doing lowk
Parts:
- moved R2 21.3 mm to (112.9, 117.0)
- moved C1 19.0 mm to (129.5, 112.5), turned to -90 degrees
- moved R1 9.51 mm to (118.1, 119.0)
- moved C3 8.71 mm to (121.5, 113.7), turned to -90 degrees
- moved L1 6.67 mm to (124.0, 108.5)
- moved C2 4.94 mm to (118.0, 108.0), turned to 0 degrees
- moved U1 2.40 mm to (118.0, 113.6), turned to -90 degrees
Routing:
- net GND: track 0.00 -> 41.5 mm
- net /VOUT: track 0.00 -> 18.5 mm
- net Net-(U1-SW): track 0.00 -> 15.8 mm
- net Net-(U1-VFB): track 0.00 -> 11.9 mm
- net +12V: track 0.00 -> 7.35 mm
- net Net-(U1-VBST): track 0.00 -> 2.71 mm
Other:
- board outline added: 21.5 x 17 mm
